File: UI基板/UI基板.kicad_pcb (KiCad board)
At the start: 2 copper layers, 12.6 x 21 mm, 15 parts, among them J1 Conn_01x04, J2 Conn_01x04, J3 Conn_01x04, U1 TFT_320x240, U2 RP2040-Zero

Commit message: ほげほげ
Parts:
- ENC1, U2: moved to B.Cu
- moved U1 194.4 mm to (242.6, 96.5), turned to 90 degrees
- moved U2 114.3 mm to (204.8, 45.9), turned to 180 degrees
- moved J3 110.0 mm to (190.6, 95.2)
- moved J2 107.9 mm to (189.2, 79.3)
- moved ENC1 61.9 mm to (147.2, 95.3), turned to 180 degrees
- moved J1 56.5 mm to (170.6, 78.5)
Connections:
- ENC1 pad 1: Net-(ENC1-RED) -> (no net)
- ENC1 pad 2: Net-(ENC1-GREEN) -> (no net)
- ENC1 pad 3: /SW -> (no net)
- ENC1 pad 4: Net-(ENC1-BLUE) -> (no net)
- ENC1 pad 5: +3.3V -> (no net)
- ENC1 pad 6: /ENC_A -> (no net)
- ENC1 pad 7: /ENC_B -> (no net)
- ENC1 pad 8: GND -> (no net)
- J1 pad 3: /RX -> /RX_in
- J1 pad 4: /TX -> /TX_in
- U2 pad 0: /TX -> /RX_in
- U2 pad 1: /RX -> /TX_in
Other:
- board size 12.6 x 21 mm -> 110 x 60 mm

Commit message: メイン基板
Parts:
- removed C2: 10u, Resistor_SMD:R_0603_1608Metric_Pad0.98x0.95mm_HandSolder
- removed J3: Conn_01x04, Connector_JST:JST_XH_S4B-XH-A_1x04_P2.50mm_Horizontal
- removed U2: RP2040-Zero, isw-kbd:RP2040-Zero-THT
- added J4: Conn_01x03, Connector_JST:JST_XH_S3B-XH-A_1x03_P2.50mm_Horizontal, B.Cu at (178.7, 82.5)
- added J5: Conn_01x04, OPL_Connector:GROVE-HW4-2.0-90D, B.Cu at (169.7, 77.8)
- added REF**: MountingHole_3.2mm_M3_DIN965_Pad, MountingHole:MountingHole_3.2mm_M3_DIN965_Pad, F.Cu at (238.1, 64.6)
- added SW1: SW_Push, Button_Switch_THT:SW_PUSH_6mm_H4.3mm, B.Cu at (189.9, 114.6)
- added SW2: ~, ハンドル基板:TTP223, F.Cu at (221.0, 68.7)
- added U3: Pico, MCU_RaspberryPi_and_Boards:RPi_Pico_SMD_TH, B.Cu at (211.9, 97.2)
- C1: value 100u -> C_Polarized_Small; moved to B.Cu
- ENC1: moved to F.Cu
- J1, R1, R2, R3: moved to B.Cu
- J2: value Conn_01x04 -> Conn_01x03; footprint Connector_JST:JST_XH_S4B-XH-A_1x04_P2.50mm_Horizontal -> Connector_JST:JST_XH_S3B-XH-A_1x03_P2.50mm_Horizontal
- moved R1 156.1 mm to (257.0, 117.0), turned to -90 degrees
- moved R2 153.0 mm to (254.5, 116.9), turned to -90 degrees
- moved C3 149.3 mm to (254.0, 95.0)
- moved R3 147.6 mm to (249.5, 117.1), turned to -90 degrees
- moved R4 147.4 mm to (254.0, 92.0), turned to 180 degrees
- moved C1 147.3 mm to (233.0, 73.7), turned to -90 degrees
- moved C4 145.5 mm to (250.5, 95.0), turned to 180 degrees
- moved R5 143.7 mm to (250.5, 92.0)
- moved ENC1 104.9 mm to (252.0, 97.6)
- moved J2 60.9 mm to (248.9, 67.0), turned to 90 degrees
- moved J1 56.9 mm to (227.3, 81.7), turned to -90 degrees
Connections:
- ENC1 pad 1: (no net) -> Net-(ENC1-RED)
- ENC1 pad 2: (no net) -> Net-(ENC1-GREEN)
- ENC1 pad 3: (no net) -> /SW
- ENC1 pad 4: (no net) -> Net-(ENC1-BLUE)
- ENC1 pad 5: (no net) -> +3.3V
- ENC1 pad 6: (no net) -> /ENC_A
- ENC1 pad 7: (no net) -> /ENC_B
- ENC1 pad 8: (no net) -> GND
- J1 pad 1: GND -> +5V
- J1 pad 2: +5V -> GND
- J1 pad 3: /RX_in -> /RX_main
- J1 pad 4: /TX_in -> /TX_main
- J2 pad 1: GND -> Net-(J2-Pin_1)
- J2 pad 2: +5V -> Net-(J2-Pin_2)
- J2 pad 3: /neopi_in -> GND
Routing:
- net /MISO: track 0.00 -> 142.2 mm
- net +5V: track 0.00 -> 126.3 mm
- net /MOSI: track 0.00 -> 110.4 mm, vias 0 -> 3
- net /SCK: track 0.00 -> 106.5 mm, vias 0 -> 6
- net +3.3V: track 0.00 -> 82.2 mm, vias 0 -> 6
- net /neopi_in: track 0.00 -> 68.8 mm, vias 0 -> 3
- net /LED_B: track 0.00 -> 55.9 mm, vias 0 -> 2
- net /CS_Touch: track 0.00 -> 49.4 mm, vias 0 -> 1
- net /ENC_A: track 0.00 -> 49.0 mm, vias 0 -> 2
- net /LED_R: track 0.00 -> 47.1 mm
- net /LED_G: track 0.00 -> 45.0 mm
- net /SW: track 0.00 -> 45.0 mm, vias 0 -> 1
- net /CS_SD: track 0.00 -> 44.1 mm, vias 0 -> 1
- net /CS_TFT: track 0.00 -> 44.0 mm, vias 0 -> 2
- net /RESET: track 0.00 -> 43.6 mm, vias 0 -> 2
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- added copper zone on B.Cu, net GND
- added copper zone on F.Cu, net GND
Other:
- board size 110 x 60 mm -> 99.5 x 64.7 mm
