File: サーボ基板/main.kicad_sch (KiCad schematic)
At the start: 13 parts, among them J10 Conn_02x10, J9 Conn_01x03, U2 DEV-16771, U3 SeeeduinoXIAO RP2040

Commit message: メイン基板
Parts:
- added C11, C12: 10u, Capacitor_THT:C_Disc_D6.0mm_W4.4mm_P5.00mm, symbol Device:C_Small
- added C13, C14, C15, C16: 0.01u, Capacitor_SMD:C_0603_1608Metric_Pad1.08x0.95mm_HandSolder, symbol Device:C_Small
- added C9: 100u, Capacitor_THT:CP_Radial_D6.3mm_P2.50mm, symbol Device:C_Polarized_Small
- added DCDC1: ~, Package_DIP:CERDIP-8_W7.62mm_SideBrazed_Socket, symbol MyLibrary:TJ7660
- added FB2, FB3: 100R, Inductor_SMD:L_Walsin_WLFM201209x, symbol Device:FerriteBead_Small
- added J11, J12, J13, J14, J15, J16: Conn_01x03_Pin, Connector_PinHeader_2.54mm:PinHeader_1x03_P2.54mm_Vertical, symbol Connector:Conn_01x03_Pin
- added J17, J18: Conn_01x05, Connector_JST:JST_XH_B5B-XH-A_1x05_P2.50mm_Vertical, symbol Connector_Generic:Conn_01x05
- added J19: Conn_01x04, Connector_JST:JST_XH_B4B-XH-A_1x04_P2.50mm_Vertical, symbol Connector_Generic:Conn_01x04
- added J20, J21: Conn_01x04, Connector_JST:JST_XH_S4B-XH-A_1x04_P2.50mm_Horizontal, symbol Connector_Generic:Conn_01x04
- added J6: Conn_01x05_Pin, Connector_PinHeader_2.54mm:PinHeader_1x05_P2.54mm_Vertical, symbol Connector:Conn_01x05_Pin
- added R10, R4, R5, R6, R7: 10k, Resistor_SMD:R_0603_1608Metric_Pad0.98x0.95mm_HandSolder, symbol Device:R_Small
- added R8, R9: 50, Resistor_SMD:R_0603_1608Metric_Pad0.98x0.95mm_HandSolder, symbol Device:R_Small
- added SW1, SW2, SW3, SW4: SW_Push, Connector_JST:JST_XH_B2B-XH-A_1x02_P2.50mm_Vertical, symbol Switch:SW_Push
- added ToF5, ToF6: ~, Connector_JST:JST_XH_B5B-XH-A_1x05_P2.50mm_Vertical, symbol ToF:VL53L1X
- added U10: SN74HC241DW, Package_DIP:CERDIP-20_W7.62mm_SideBrazed_Socket, symbol 2024-09-28_15-43-53:SN74HC241DW
- added U4, U5: AD8226ARZ, MyLibrary:SOP-8_DIP, symbol 2024-09-28_14-00-08:AD8226ARZ
- added U8, U9: ADuM121N, MyLibrary:SOP-8_DIP, symbol Isolator:ADuM121N
- FL1: footprint BNX012H01_MUR -> BNX012-01:BNX012H01_MUR
- Gyro1: footprint (none) -> MyLibrary:BNO055
Connections:
- net +5VA: now also C9.1, FB3.2, J11.2 (Pin_2), J12.2 (Pin_2), J13.2 (Pin_2), J14.2 (Pin_2), J15.2 (Pin_2), J16.2 (Pin_2), J17.4 (Pin_4), J18.4 (Pin_4), J19.1 (Pin_1), ToF5.1 (VIN), ToF6.1 (VIN)
- net +5VD: now also J6.5 (Pin_5)
- net GND2: now also C12.1, C13.2, C15.2, C9.2, DCDC1.3 (GND), J11.1 (Pin_1), J12.1 (Pin_1), J13.1 (Pin_1), J14.1 (Pin_1), J15.1 (Pin_1), J16.1 (Pin_1), J17.5 (Pin_5), J18.5 (Pin_5), J19.2 (Pin_2), J20.4 (Pin_4), J21.4 (Pin_4), J6.4 (Pin_4), R4.2, R5.2, R6.2, R7.2, ToF5.2 (GND), ToF6.2 (GND), U4.6 (REF), U5.6 (REF), U8.4 (GND1), U9.4 (GND1)
- net Line1: now also U2.41 (A17); no longer U2.23 (A9)
- net Line11: now also U2.39 (A15); no longer U2.27 (A13)
- net Line2: now also U2.40 (A16); no longer U2.22 (A8)
- net Line3: now also U2.14 (A0); no longer U2.21 (A7)
- net Line4: now also U2.15 (A1); no longer U2.20 (A6)
- net Line5: now also U2.20 (A6); no longer U2.15 (A1)
- net Line6: now also U2.21 (A7); no longer U2.14 (A0)
- net Line7: now also U2.22 (A8); no longer U2.41 (A17)
- net Line8: now also U2.23 (A9); no longer U2.40 (A16)
- net Line9: now also U2.27 (A13); no longer U2.39 (A15)
- net PWM1: now also J11.3 (Pin_3)
- net PWM2: now also J12.3 (Pin_3)
- net PWM3: now also J13.3 (Pin_3)
- net PWM4: now also J14.3 (Pin_3)
- net PWM5: now also J15.3 (Pin_3)
- net PWM6: now also J16.3 (Pin_3)
- net loadcell1: now also U4.7 (VOUT)
- net loadcell2: now also U5.7 (VOUT)
- net rx_dxl: now also U9.2 (VOA)
- net scl: now also ToF5.4 (SCL), ToF6.4 (SCL)
- net scl_sub: now also J17.2 (Pin_2), J18.2 (Pin_2)
- net sda: now also ToF5.3 (SDA), ToF6.3 (SDA)
- net sda_sub: now also J17.3 (Pin_3), J18.3 (Pin_3)
- net tx_dxl: now also U9.3 (VIB)
- net tx_en: now also U2.2 (OUT2), U8.3 (VIB); no longer U2.5 (IN2)
- net xshut1: now also U2.6 (OUT1D); no longer U2.2 (OUT2)
- net xshut2: now also U2.9 (OUT1C); no longer ToF1.5 (XSHUT), U2.3 (LRCLK2)
- net xshut3: now also ToF1.5 (XSHUT); no longer ToF2.5 (XSHUT)
- net xshut4: now also U2.5 (IN2); no longer U2.6 (OUT1D)
- net xshut5: now also ToF2.5 (XSHUT), U2.10 (CS1); no longer ToF4.5 (XSHUT), U2.7 (RX2)
- net xshut6: now also ToF4.5 (XSHUT), U2.3 (LRCLK2); no longer U2.8 (TX2)
- net xshut7: now also U2.11 (MOSI), ToF5.5 (XSHUT); no longer U2.9 (OUT1C)
- net xshut8: now also U2.12 (MISO), ToF6.5 (XSHUT); no longer U2.10 (CS1)
- net rx_main_power: now reaches U2.25 (A11)
- net rx_main_power: now also U8.2 (VOA)
- net +3.3V: now reaches U2.3.3V_2 (3.3V)
- net +3.3V: now also DCDC1.8 (V+), J20.1 (Pin_1), J21.1 (Pin_1), SW1.1, SW2.1, SW3.1, SW4.1, U4.8 (VS+), U5.8 (VS+)
- net LimSW1: now reaches U2.30 (CRX3)
- net LimSW1: now also R4.1, SW1.2
- net LimSW2: now reaches U2.31 (CTX3)
- net LimSW2: now also R5.1, SW2.2
- net LimSW3: now reaches U2.32 (OUT1B)
- net LimSW3: now also R6.1, SW3.2
- net LimSW4: now reaches U2.33 (MCLK2)
- net LimSW4: now also R7.1, SW4.2
- net xshut_sub: now reaches U3.11 (PA6_A10_D10_MOSI)
- net xshut_sub: now also J18.1 (Pin_1)
- net LiDAR_TX: now reaches Pi1.10 (GPIO15/RXD0)
- net LiDAR_TX: now also J6.1 (Pin_1)
- net LiDAR_PWM: now reaches Pi1.12 (GPIO18/GPIO_GEN1)
- net LiDAR_PWM: now also J6.2 (Pin_2)
- new net: C13.1, C15.1, FB3.1, U8.1 (VDD1), U9.1 (VDD1)
- new net: U10.1 (*1OE), U10.19 (2OE), U8.6 (VOB)
- new net: U10.17 (2A4), U9.6 (VOB)
- new net: U10.18 (1Y1), U9.7 (VIA)
- new net: C14.1, C16.2, FB2.2, U8.8 (VDD2), U9.8 (VDD2)
- new net: R9.1, U5.2 (RG)
- new net: R9.2, U5.3 (RG)
- new net: C11.1, DCDC1.2 (CAP+)
- new net: C11.2, DCDC1.4 (CAP-)
- new net: R8.1, U4.2 (RG)
- new net: R8.2, U4.3 (RG)
- new net +5V: FB2.1, R10.2, U10.20 (VCC)
- new net DATA: R10.1, U10.2 (1A1), U10.3 (2Y4)
- new net GND: C14.2, C16.1, U10.10 (GND), U8.5 (GND2), U9.5 (GND2)
- new net LdCl_GREEN1: J20.3 (Pin_3), U4.4 (IN+)
- new net LdCl_GREEN2: J21.3 (Pin_3), U5.4 (IN+)
- new net LdCl_WHITE1: J20.2 (Pin_2), U4.1 (IN-)
- new net LdCl_WHITE2: J21.2 (Pin_2), U5.1 (IN-)
- new net RX_Main_Power_Sub: U8.7 (VIA)
- new net VEE: C12.2, DCDC1.5 (VOUT), U4.5 (VS-), U5.5 (VS-)
- new net rx2_main: J19.3 (Pin_3), U2.7 (RX2)
- new net tx2_main: J19.4 (Pin_4), U2.8 (TX2)
- no-connect marks 55 -> 73
Other:
- note added: "I2C RESETを飛ばすこと!"
- note added: "LiDAR"
- note added: "PWMサーボ"
- note added: "UI"
- note added: "VL53L1X"
- note added: "VL53L5CX"
- note added: "サブマイコン"
- note added: "シリアル変換+アイソレート"
- note added: "リミットスイッチ"
- note added: "ロードセル"
- moved on the sheet: FL1, Gyro1, J10, J9, Pi1, ToF1, ToF2, ToF3, ToF4, U3
