File: サーボ基板/サーボ基板.kicad_pcb (KiCad board)
At the start: 2 copper layers, 76.2 x 59.7 mm, 26 parts, among them J1 Conn_01x02, J2 Conn_01x03, J3 Conn_01x03, J4 Conn_01x03, J5 Conn_01x03, J6 DATA_IN, U1 SeeeduinoXIAO RP2040

Commit message: サーボ基板
Parts:
- removed ? (x3): , 
- removed the REF** at (43.2, 94.0)
- added ENC1: ~, Potentiometer_LED:EC12PLRGBSDVBF, F.Cu at (208.9, 110.2)
- added J7: Conn_01x05_Pin, Connector_PinHeader_2.54mm:PinHeader_1x05_P2.54mm_Vertical, F.Cu at (198.1, 115.3)
- added J8: Conn_01x03_Pin, Connector_PinHeader_2.54mm:PinHeader_1x03_P2.54mm_Vertical, F.Cu at (221.0, 112.8)
- added REF**: MountingHole_3.2mm_M3_DIN965_Pad, MountingHole:MountingHole_3.2mm_M3_DIN965_Pad, F.Cu at (101.6, 79.4)
- added REF**: MountingHole_3.2mm_M3_DIN965_Pad, MountingHole:MountingHole_3.2mm_M3_DIN965_Pad, F.Cu at (59.7, 79.4)
- added REF**: MountingHole_3.2mm_M3_DIN965_Pad, MountingHole:MountingHole_3.2mm_M3_DIN965_Pad, F.Cu at (84.5, 79.4)
- D1: footprint LED_THT:LED_D5.0mm_Horizontal_O1.27mm_Z3.0mm -> LED_THT:LED_D5.0mm
- J1: moved to B.Cu
- moved J5 71.0 mm to (39.8, 68.0), turned to -90 degrees
- moved C10 67.4 mm to (40.7, 64.0), turned to 0 degrees
- moved J4 63.4 mm to (45.7, 68.0), turned to -90 degrees
- moved J1 62.6 mm to (44.8, 85.9), turned to 0 degrees
- moved C8 60.4 mm to (46.6, 64.0), turned to 0 degrees
- moved J3 56.1 mm to (51.5, 68.0), turned to -90 degrees
- moved U1 55.0 mm to (101.6, 88.9), turned to 0 degrees
- moved C6 52.0 mm to (52.4, 64.0), turned to 0 degrees
- moved C5 49.3 mm to (46.5, 78.6), turned to -90 degrees
- moved J2 49.0 mm to (57.4, 68.0), turned to -90 degrees
- moved C3 45.2 mm to (58.2, 64.0), turned to 0 degrees
- moved R3 45.1 mm to (91.5, 90.0), turned to 90 degrees
- moved R2 45.0 mm to (98.5, 85.1), turned to 0 degrees
- moved R1 43.8 mm to (97.6, 88.1), turned to 90 degrees
- moved J6 31.8 mm to (63.8, 66.0)
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Connections:
- D1 pad 1: Net-(D1-K) -> GND
- D1 pad 2: /RED LED -> Net-(D1-A)
- R3 pad 1: Net-(D1-K) -> /RED LED
- R3 pad 2: GND -> Net-(D1-A)
Routing:
- net Net-(D1-A): track 0.00 -> 54.7 mm, vias 0 -> 2
- net VDD: track 125.0 -> 88.5 mm, vias 1 -> 0
- net Net-(J4-Pin_2): track 85.5 -> 53.7 mm
- net Net-(U1-PA02_A0_D0): track 20.1 -> 6.93 mm, vias 0 -> 1
- net /DCDC RST1: track 43.7 -> 31.3 mm, vias 3 -> 0
- net Net-(D1-K): track 6.62 -> 0.00 mm
- net Net-(J2-Pin_2): track 61.3 -> 55.5 mm
- net /DATA: track 34.4 -> 29.4 mm
- net Net-(ENC1-A): track 0.00 -> 4.62 mm
- net Net-(ENC1-C): track 0.00 -> 4.62 mm
- net Net-(ENC1-B): track 0.00 -> 4.55 mm
- net Net-(ENC1-RED): track 0.00 -> 4.27 mm
- net Net-(ENC1-Anode): track 0.00 -> 4.26 mm
- net Net-(ENC1-GREEN): track 0.00 -> 4.04 mm
- net Net-(ENC1-BLUE): track 0.00 -> 4.03 mm
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Other:
- board size 76.2 x 59.7 mm -> 188 x 54.4 mm
- board text removed: "DXL1"
- board text removed: "DXL2"
- board text removed: "DXL3"
- board text removed: "DXL4"

Commit message: メイン基板
Parts:
- removed ENC1: ~, Potentiometer_LED:EC12PLRGBSDVBF
- removed J7: Conn_01x05_Pin, Connector_PinHeader_2.54mm:PinHeader_1x05_P2.54mm_Vertical
- removed J8: Conn_01x03_Pin, Connector_PinHeader_2.54mm:PinHeader_1x03_P2.54mm_Vertical
- removed the REF** at (101.6, 79.4)
- removed the REF** at (59.7, 79.4)
- removed the REF** at (84.5, 79.4)
- added ?: , , F.Cu at (52.7, 103.9)
- added ?: , , F.Cu at (101.7, 161.9)
- added ?: , , F.Cu at (52.7, 161.9)
- added C11: 10u, Capacitor_THT:C_Disc_D6.0mm_W4.4mm_P5.00mm, F.Cu at (128.8, 61.2)
- added C12: 10u, Capacitor_THT:C_Disc_D6.0mm_W4.4mm_P5.00mm, F.Cu at (128.9, 41.6)
- added C13: 0.01u, Capacitor_SMD:C_0603_1608Metric_Pad1.08x0.95mm_HandSolder, F.Cu at (100.6, 58.4)
- added C14: 0.01u, Capacitor_SMD:C_0603_1608Metric_Pad1.08x0.95mm_HandSolder, B.Cu at (97.1, 48.4)
- added C15: 0.01u, Capacitor_SMD:C_0603_1608Metric_Pad1.08x0.95mm_HandSolder, F.Cu at (90.2, 58.4)
- added C16: 0.01u, Capacitor_SMD:C_0603_1608Metric_Pad1.08x0.95mm_HandSolder, B.Cu at (89.9, 48.2)
- added C7: 100u, Capacitor_THT:CP_Radial_D6.3mm_P2.50mm, F.Cu at (109.9, 179.1)
- added C9: 100u, Capacitor_THT:CP_Radial_D6.3mm_P2.50mm, F.Cu at (82.6, 22.9)
- added DCDC1: ~, Package_DIP:CERDIP-8_W7.62mm_SideBrazed_Socket, F.Cu at (130.2, 55.3)
- added FB1: 100R, Inductor_SMD:L_Walsin_WLFM201209x, F.Cu at (111.5, 185.0)
- added FB2: 100R, Inductor_SMD:L_Walsin_WLFM201209x, B.Cu at (97.2, 50.2)
- added FB3: 100R, Inductor_SMD:L_Walsin_WLFM201209x, F.Cu at (77.5, 58.4)
- added FL1: BNX012-01, BNX012-01:BNX012H01_MUR, F.Cu at (86.4, 160.6)
- added G***: LOGO, logo:logo, F.Cu at (125.1, 94.3)
- added Gyro1: ~, MyLibrary:BNO055, F.Cu at (41.3, 163.2)
- added J10: Conn_02x10, Connector_PinHeader_2.54mm:PinHeader_2x10_P2.54mm_Vertical, F.Cu at (77.5, 69.8)
- added J11: Conn_01x03_Pin, Connector_PinHeader_2.54mm:PinHeader_1x03_P2.54mm_Vertical, F.Cu at (36.2, 45.7)
- added J12: Conn_01x03_Pin, Connector_PinHeader_2.54mm:PinHeader_1x03_P2.54mm_Vertical, F.Cu at (40.0, 45.7)
- added J13: Conn_01x03_Pin, Connector_PinHeader_2.54mm:PinHeader_1x03_P2.54mm_Vertical, F.Cu at (43.8, 45.7)
- added J14: Conn_01x03_Pin, Connector_PinHeader_2.54mm:PinHeader_1x03_P2.54mm_Vertical, F.Cu at (47.6, 45.7)
- added J15: Conn_01x03_Pin, Connector_PinHeader_2.54mm:PinHeader_1x03_P2.54mm_Vertical, F.Cu at (43.1, 179.1)
- added J16: Conn_01x03_Pin, Connector_PinHeader_2.54mm:PinHeader_1x03_P2.54mm_Vertical, F.Cu at (38.7, 179.1)
- added J17: Conn_01x05, Connector_JST:JST_XH_B5B-XH-A_1x05_P2.50mm_Vertical, F.Cu at (114.9, 24.8)
- added J18: Conn_01x05, Connector_JST:JST_XH_B5B-XH-A_1x05_P2.50mm_Vertical, F.Cu at (52.6, 33.7)
- added J19: Conn_01x04, Connector_JST:JST_XH_B4B-XH-A_1x04_P2.50mm_Vertical, F.Cu at (138.4, 150.6)
- added J20: Conn_01x04, Connector_JST:JST_XH_S4B-XH-A_1x04_P2.50mm_Horizontal, B.Cu at (75.9, 97.3)
- added J21: Conn_01x04, Connector_JST:JST_XH_S4B-XH-A_1x04_P2.50mm_Horizontal, B.Cu at (89.9, 97.3)
- added J9: Conn_01x03, Connector_JST:JST_VH_B3PS-VH_1x03_P3.96mm_Horizontal, B.Cu at (80.0, 168.3)
- added Pi1: RASPBERRY_PI_4B_4GB, Raspberry Pi 5:Raspberry Pi 5, F.Cu at (109.9, 133.0)
- added R10: 10k, Resistor_SMD:R_0603_1608Metric_Pad0.98x0.95mm_HandSolder, F.Cu at (59.1, 56.5)
- added R4: 10k, Resistor_SMD:R_0603_1608Metric_Pad0.98x0.95mm_HandSolder, F.Cu at (47.6, 35.1)
- added R5: 10k, Resistor_SMD:R_0603_1608Metric_Pad0.98x0.95mm_HandSolder, F.Cu at (124.0, 35.6)
- added R6: 10k, Resistor_SMD:R_0603_1608Metric_Pad0.98x0.95mm_HandSolder, F.Cu at (46.1, 183.0)
- added R7: 10k, Resistor_SMD:R_0603_1608Metric_Pad0.98x0.95mm_HandSolder, F.Cu at (110.1, 161.2)
- added R8: 50, Resistor_SMD:R_0603_1608Metric_Pad0.98x0.95mm_HandSolder, F.Cu at (107.8, 43.8)
- added R9: 50, Resistor_SMD:R_0603_1608Metric_Pad0.98x0.95mm_HandSolder, F.Cu at (108.0, 55.9)
- added REF**: MountingHole_3.2mm_M3_DIN965_Pad, MountingHole:MountingHole_3.2mm_M3_DIN965_Pad, F.Cu at (136.5, 165.1)
- added REF**: MountingHole_2.5mm, MountingHole:MountingHole_2.5mm, F.Cu at (101.7, 103.9)
- added REF**: MountingHole_3.2mm_M3_DIN965_Pad, MountingHole:MountingHole_3.2mm_M3_DIN965_Pad, F.Cu at (136.5, 47.0)
- added REF**: MountingHole_3.2mm_M3_DIN965_Pad, MountingHole:MountingHole_3.2mm_M3_DIN965_Pad, F.Cu at (31.1, 165.1)
- added REF**: MountingHole_3.2mm_M3_DIN965_Pad, MountingHole:MountingHole_3.2mm_M3_DIN965_Pad, F.Cu at (31.1, 47.0)
- added SW1: SW_Push, Connector_JST:JST_XH_B2B-XH-A_1x02_P2.50mm_Vertical, F.Cu at (45.3, 30.2)
- added SW2: SW_Push, Connector_JST:JST_XH_B2B-XH-A_1x02_P2.50mm_Vertical, F.Cu at (121.0, 30.5)
- added SW3: SW_Push, Connector_JST:JST_XH_B2B-XH-A_1x02_P2.50mm_Vertical, F.Cu at (39.8, 183.9)
- added SW4: SW_Push, Connector_JST:JST_XH_B2B-XH-A_1x02_P2.50mm_Vertical, F.Cu at (109.2, 168.5)
- added ToF1: ~, ToF:GY530, F.Cu at (31.8, 30.5)
- added ToF2: ~, ToF:GY530, F.Cu at (135.9, 30.5)
- added ToF3: ~, ToF:GY530, F.Cu at (31.8, 181.6)
- added ToF4: ~, ToF:GY530, F.Cu at (135.9, 181.6)
- added ToF5: ~, Connector_JST:JST_XH_B5B-XH-A_1x05_P2.50mm_Vertical, F.Cu at (128.3, 35.5)
- added ToF6: ~, Connector_JST:JST_XH_B5B-XH-A_1x05_P2.50mm_Vertical, F.Cu at (39.2, 25.4)
- added U10: SN74HC241DW, Package_DIP:CERDIP-20_W7.62mm_SideBrazed_Socket, B.Cu at (52.7, 46.4)
- added U2: DEV-16771, DEV-16771:MODULE_DEV-16771, F.Cu at (123.2, 155.8)
- added U3: SeeeduinoXIAO RP2040, XIAO RP2040:XIAO RP2040, B.Cu at (83.8, 30.5)
- added U4: AD8226ARZ, MyLibrary:SOP-8_DIP, F.Cu at (114.2, 43.8)
- added U5: AD8226ARZ, MyLibrary:SOP-8_DIP, F.Cu at (114.2, 55.9)
- added U8: ADuM121N, MyLibrary:SOP-8_DIP, B.Cu at (95.9, 50.2)
- added U9: ADuM121N, MyLibrary:SOP-8_DIP, B.Cu at (83.8, 50.2)
- J2, J3: footprint Connector_JST:JST_EH_B3B-EH-A_1x03_P2.50mm_Vertical -> Connector_JST:JST_EH_S3B-EH_1x03_P2.50mm_Horizontal; moved to B.Cu
- J6: value DATA_IN -> Conn_01x05_Pin; footprint Connector_JST:JST_XH_B2B-XH-A_1x02_P2.50mm_Vertical -> Connector_PinHeader_2.54mm:PinHeader_1x05_P2.54mm_Vertical
- moved J6 77.0 mm to (117.1, 121.5), turned to 180 degrees
- moved R3 70.6 mm to (30.3, 54.7), turned to 180 degrees
- moved U1 67.8 mm to (41.7, 57.3), turned to 180 degrees
- moved R1 63.3 mm to (35.1, 78.6)
- moved R2 57.1 mm to (45.5, 64.0), turned to 90 degrees
- moved C2 47.7 mm to (42.6, 54.0), turned to 180 degrees
- moved C4 36.1 mm to (29.5, 67.7)
- moved LDO1 32.4 mm to (62.2, 60.6), turned to 180 degrees
- moved LT1 30.6 mm to (59.7, 67.3), turned to -90 degrees
- moved C1 29.2 mm to (66.0, 63.5)
- moved D1 21.8 mm to (29.5, 60.1), turned to 90 degrees
- moved C10 21.0 mm to (39.6, 85.0)
- moved C3 15.2 mm to (43.4, 67.4), turned to 180 degrees
- moved C8 13.8 mm to (48.5, 77.6), turned to -90 degrees
- moved J5 13.3 mm to (39.4, 81.3), turned to 0 degrees
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Connections:
- J2 pad 3: /DATA -> DATA
- J3 pad 3: /DATA -> DATA
- J4 pad 3: /DATA -> DATA
- J5 pad 3: /DATA -> DATA
- J6 pad 1: GND -> /main/LiDAR_TX
- J6 pad 2: /DATA -> /main/LiDAR_PWM
- U1 pad 6: /GREEN LED -> unconnected-(U1-PA9_A5_D5_SCL-Pad6)
- U1 pad 7: unconnected-(U1-PB08_A6_D6_TX-Pad7) -> RX_Main_Power_Sub
Routing:
- net +5VA: track 0.00 -> 563.8 mm, vias 0 -> 3
- net /main/sda: track 0.00 -> 426.0 mm, vias 0 -> 7
- net /main/scl: track 0.00 -> 425.1 mm, vias 0 -> 13
- net +3.3V: track 0.00 -> 401.6 mm, vias 0 -> 8
- net /main/xshut3: track 0.00 -> 229.5 mm, vias 0 -> 2
- net /main/xshut8: track 0.00 -> 216.9 mm, vias 0 -> 4
- net /main/LimSW1: track 0.00 -> 216.3 mm, vias 0 -> 3
- net /main/PWM6: track 0.00 -> 210.2 mm
- net /main/PWM5: track 0.00 -> 208.3 mm
- net /main/loadcell1: track 0.00 -> 181.9 mm, vias 0 -> 4
- net /main/loadcell2: track 0.00 -> 162.4 mm, vias 0 -> 7
- net /main/tx_dxl: track 0.00 -> 160.0 mm, vias 0 -> 5
- net /main/rx_dxl: track 0.00 -> 158.5 mm, vias 0 -> 3
- net /main/tx_en: track 0.00 -> 147.5 mm, vias 0 -> 4
- net /main/Line8: track 0.00 -> 147.3 mm, vias 0 -> 3
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- added copper zone on B.Cu, net GND2
- added copper zone on F.Cu, net GND2
Other:
- board size 188 x 54.4 mm -> 120 x 170.1 mm
