File: ライン基板/ライン基板.kicad_pcb (KiCad board)
At the start: 2 copper layers, 99.6 x 61.6 mm, 50 parts, among them J1 Conn_02x10, J2 Conn_01x06, J3 ColorSensor, J4 ColorSensor, J5 Conn_01x06

Commit message: メイン基板
Parts:
- added ENC1: ~, Potentiometer_LED:EC12PLRGBSDVBF, F.Cu at (105.4, 42.4)
- added J1: Conn_01x05_Pin, Connector_PinHeader_2.54mm:PinHeader_1x05_P2.54mm_Vertical, F.Cu at (94.6, 47.5)
- added J2: Conn_01x03_Pin, Connector_PinHeader_2.54mm:PinHeader_1x03_P2.54mm_Vertical, F.Cu at (117.4, 44.9)
Connections:
- J4 pad 8: GND2 -> GND
- J5 pad 2: GND2 -> GND
- ToF1 pad 6: GND2 -> GND
- ToF2 pad 6: GND2 -> GND
- color1 pad 1: GND2 -> GND
- color2 pad 1: GND2 -> GND
Routing:
- net (no net): track 0.00 -> 34.1 mm
- net GND: track 0.00 -> 12.3 mm, vias 191 -> 234
- net GND2: vias 43 -> 0
- removed copper zone on B.Cu, net GND2
- removed copper zone on F.Cu, net GND2
Other:
- board size 99.6 x 61.6 mm -> 99.6 x 77 mm
