File: ライン基板/ライン基板.kicad_sch (KiCad schematic)
At the start: 48 parts, among them J1 Conn_02x10, J2 Conn_01x06, J3 ColorSensor, J4 ColorSensor, J5 Conn_01x06

Commit message: メイン基板
Connections:
- net GND2 is gone; now on net GND: J4.8 (Pin_8), J5.2 (Pin_2), ToF1.6 (GND), ToF2.6 (GND), color1.1 (GND), color2.1 (GND)
Changed lines of the file:
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@@
 	)
 	(junction
+		(at 232.41 36.83)
+		(diameter 0)
+		(color 0 0 0 0)
+	)
+	(junction
 		(at 110.49 44.45)
 		(diameter 0)
@@
 					(unit 1)
 				)
+			)
+		)
+	)
+	(symbol
+		(lib_id "power:GND")
+		(at 232.41 36.83 180)
+		(unit 1)
+		(exclude_from_sim no)
+		(in_bom yes)
+		(on_board yes)
+		(dnp no)
+		(fields_autoplaced yes)
+		(property "Reference" "#PWR07"
+			(at 232.41 30.48 0)
+			(effects
+				(font
+					(size 1.27 1.27)
+				)
+				(hide yes)
+			)
+		)
+		(property "Value" "GND"
+			(at 232.41 31.75 0)
+			(effects
+				(font
+					(size 1.27 1.27)
+				)
+			)
+		)
+		(property "Footprint" ""
+			(at 232.41 36.83 0)
+			(effects
+				(font
+					(size 1.27 1.27)
+				)
+				(hide yes)
+			)
+		)
+		(property "Datasheet" ""
+			(at 232.41 36.83 0)
+			(effects
+				(font
+					(size 1.27 1.27)
+				)
+				(hide yes)
+			)
+		)
+		(property "Description" "Power symbol creates a global label with name \"GND\" , ground"
+			(at 232.41 36.83 0)
+			(effects
+				(font
+					(size 1.27 1.27)
+				)
+				(hide yes)
+			)
+		)
+		(pin "1"
+		)
+		(instances
+			(project "ライン基板"
+				(path "/97bdc067-c308-49c6-a617-dc8fcf84b17f"
+					(reference "#PWR07")
+					(unit 1)
+				)
