File: Sub/Sub.kicad_sch (KiCad schematic)
At the start: 26 parts, among them J2 Conn_01x03_Pin, J3 Conn_01x03_Pin, J4 Conn_01x03_Pin, J5 Conn_01x03_Pin, J6 Conn_01x05, J7 Conn_01x05, J8 Conn_01x04, J9 Conn_01x04, SW1 SW_Push, SW2 SW_Push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

Commit message: 電源基板にATtiny用LDOを追加
Parts:
- removed C1: 100u, Capacitor_THT:CP_Radial_D6.3mm_P2.50mm, symbol Device:C_Polarized_Small
- removed U1: SeeeduinoXIAO RP2040, XIAO RP2040:XIAO RP2040, symbol Seeeduino XIAO:SeeeduinoXIAO
- added C4: C_Polarized_Small, Capacitor_THT:CP_Radial_D5.0mm_P2.50mm, symbol Device:C_Polarized_Small
- added SW3: SW_Push, Button_Switch_THT:SW_PUSH_6mm_H4.3mm, symbol Switch:SW_Push
- added ToF5: ~, ToF:GY530, symbol ToF:GY530
- added U4: Pico, RPi_Pico:RPi_Pico_SMD_TH, symbol MCU_RaspberryPi_and_Boards:Pico
Connections:
- net +3.3V: now also U4.36 (3V3)
- net +5VA: now also C4.2, ToF5.1 (VIN), U4.39 (VSYS)
- net GND2: now also C4.1, ToF5.2 (GND), U4.13 (GND), U4.18 (GND), U4.23 (GND), U4.28 (GND), U4.3 (GND), U4.38 (GND), U4.8 (GND)
- net PWM1: now also U4.14 (GPIO10)
- net PWM2: now also U4.15 (GPIO11)
- net PWM3: now also U4.16 (GPIO12)
- net PWM4: now also U4.17 (GPIO13)
- net PWM5: now also U4.19 (GPIO14)
- net PWM6: now also U4.20 (GPIO15)
- net rx8_main: now also U4.1 (GPIO0)
- net rx_sub: now also U4.2 (GPIO1)
- net scl_sub: now also ToF5.3 (SCL), U4.7 (GPIO5)
- net sda_sub: now also ToF5.4 (SDA), U4.6 (GPIO4)
- net tx: now also U4.5 (GPIO3)
- net xshut1_sub: now reaches J6.1 (Pin_1)
- net xshut1_sub: now also U4.10 (GPIO7)
- net xshut_sub renamed xshut2_sub
- net xshut2_sub: now also U4.11 (GPIO8)
- new net CS: U4.22 (GPIO17)
- new net GND: SW3.2
- new net MISO: U4.21 (GPIO16)
- new net MOSI: U4.25 (GPIO19)
- new net SCK: U4.24 (GPIO18)
- new net enable_pico: SW3.1, U4.30 (RUN)
- new net xshut3_sub: ToF5.5 (XSHUT), U4.12 (GPIO9)
Other:
- note added: "Pico 2"
- note removed: "XIAO RP2040"
- moved on the sheet: J6, J7, ToF3, ToF4
